File: PCB/Rev1.2-socket-left/ergodash.kicad_sch (KiCad schematic)
At the start: 81 parts, among them J1 5PIN, SW1 SW_PUSH, SW10 SW_PUSH, SW11 SW_PUSH, SW12 SW_PUSH, SW13 SW_PUSH, SW14 SW_PUSH, SW15 SW_PUSH, SW16 SW_PUSH, SW17 SW_PUSH, SW18 SW_PUSH, SW19 SW_PUSH, SW2 SW_PUSH, SW20 SW_PUSH, SW21 SW_PUSH, SW22 SW_PUSH, SW23 SW_PUSH, SW24 SW_PUSH, SW25 SW_PUSH, SW26 SW_PUSH, SW27 SW_PUSH, SW28 SW_PUSH, SW29 SW_Push, SW3 SW_PUSH, SW30 SW_PUSH, SW31 SW_PUSH, SW32 SW_PUSH, SW33 SW_PUSH, SW34 SW_PUSH, SW35 SW_PUSH, SW4 SW_PUSH, SW40 SW_PUSH, SW5 SW_PUSH, SW6 SW_PUSH, SW7 SW_PUSH, SW8 SW_PUSH, SW9 SW_PUSH, U1 HOLE, U2 HOLE, U3 ProMicro, U4 HOLE, U5 HOLE, U6 ProMicro, U7 HOLE, U8 HOLE, U9 HOLE

Commit message: Remove vestigial U6, add Pro Micro pin labels, refresh both boards
Schematic cleanup: delete U6 (the right-hand Pro Micro left over from the
original reversible design) from both halves' schematics. It was on_board=no
so it never appeared in the netlist or on the board; removing it just drops
dead symbols. Both schematics remain electrically identical.

Left board: add silkscreen pin-name labels (RAW/GND/RST/VCC/TX0/RX1...) around
the Pro Micro, and stamp the title block as Socket-left.

Right board: re-mirror from the left so it inherits the new pin labels and is
stamped Socket-right (mirror_right.py now swaps the title). Regenerate gerbers
and drill for both halves.

DRC: left 130 / right 131 violations (all pre-existing cosmetic/library items,
down from 137), schematic-parity 0, unrouted 0.

Co-Authored-By: Claude Opus 4.8 <noreply@anthropic.com>
Parts:
- removed U6: ProMicro, library:ProMicro_rev, symbol promicro:ProMicro
Connections:
- no-connect marks 2 -> 1
